File: 2022-09-26_termostato_kicad6/termostato_kicad6/termostato_kicad6.kicad_sch (KiCad schematic)
At the start: 13 parts, among them K1 SRD-05VDC-SL-C, Q1 BC337, U1 MCP6002-xP, X1 Power 5V, X2 OUT

Commit message: layout
Parts:
- added H1, H2, H3, H4: MountingHole, MountingHole:MountingHole_4.3mm_M4, symbol Mechanical:MountingHole
Changed lines of the file:
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@@
     (pin "1")
+  )
+  (symbol (lib_id "Mechanical:MountingHole") (at 184.15 158.75 0) (unit 1)
+    (in_bom yes) (on_board yes) (fields_autoplaced)
+    (property "Reference" "H3" (id 0) (at 186.69 158.7499 0)
+      (effects (font (size 1.27 1.27)) (justify left))
+    )
+    (property "Value" "MountingHole" (id 1) (at 186.69 160.0199 0)
+      (effects (font (size 1.27 1.27)) (justify left) hide)
+    )
+    (property "Footprint" "MountingHole:MountingHole_4.3mm_M4" (id 2) (at 184.15 158.75 0)
+      (effects (font (size 1.27 1.27)) hide)
+    )
+    (property "Datasheet" "~" (id 3) (at 184.15 158.75 0)
+      (effects (font (size 1.27 1.27)) hide)
+    )
+  )
+  (symbol (lib_id "Mechanical:MountingHole") (at 193.04 158.75 0) (unit 1)
+    (in_bom yes) (on_board yes) (fields_autoplaced)
+    (property "Reference" "H4" (id 0) (at 195.58 158.7499 0)
+      (effects (font (size 1.27 1.27)) (justify left))
+    )
+    (property "Value" "MountingHole" (id 1) (at 195.58 160.0199 0)
+      (effects (font (size 1.27 1.27)) (justify left) hide)
+    )
+    (property "Footprint" "MountingHole:MountingHole_4.3mm_M4" (id 2) (at 193.04 158.75 0)
+      (effects (font (size 1.27 1.27)) hide)
+    )
+    (property "Datasheet" "~" (id 3) (at 193.04 158.75 0)
+      (effects (font (size 1.27 1.27)) hide)
+    )
   )
   (symbol (lib_id "Amplifier_Operational:MCP6002-xP") (at 125.73 95.25 0) (unit 1)
@@
     (pin "8")
   )
+  (symbol (lib_id "Mechanical:MountingHole") (at 184.15 153.67 0) (unit 1)
+    (in_bom yes) (on_board yes) (fields_autoplaced)
+    (property "Reference" "H1" (id 0) (at 186.69 153.6699 0)
+      (effects (font (size 1.27 1.27)) (justify left))
+    )
+    (property "Value" "MountingHole" (id 1) (at 186.69 154.9399 0)
+      (effects (font (size 1.27 1.27)) (justify left) hide)
+    )
+    (property "Footprint" "MountingHole:MountingHole_4.3mm_M4" (id 2) (at 184.15 153.67 0)
+      (effects (font (size 1.27 1.27)) hide)
+    )
+    (property "Datasheet" "~" (id 3) (at 184.15 153.67 0)
+      (effects (font (size 1.27 1.27)) hide)
+    )
+  )
   (symbol (lib_id "Amplifier_Operational:MCP6002-xP") (at 179.07 96.52 0) (unit 2)
     (in_bom yes) (on_board yes) (fields_autoplaced)
@@
     (pin "2")
   )
+  (symbol (lib_id "Mechanical:MountingHole") (at 193.04 153.67 0) (unit 1)
+    (in_bom yes) (on_board yes) (fields_autoplaced)
+    (property "Reference" "H2" (id 0) (at 195.58 153.6699 0)
+      (effects (font (size 1.27 1.27)) (justify left))
+    )
+    (property "Value" "MountingHole" (id 1) (at 195.58 154.9399 0)
+      (effects (font (size 1.27 1.27)) (justify left) hide)
+    )
+    (property "Footprint" "MountingHole:MountingHole_4.3mm_M4" (id 2) (at 193.04 153.67 0)
+      (effects (font (size 1.27 1.27)) hide)
+    )
+    (property "Datasheet" "~" (id 3) (at 193.04 153.67 0)
+      (effects (font (size 1.27 1.27)) hide)
+    )
+  )
   (symbol (lib_id "Device:R") (at 110.49 92.71 90) (unit 1)
     (in_bom yes) (on_board yes) (fields_autoplaced)
@@
       (reference "D1") (unit 1) (value "1N4004") (footprint "Diode_THT:D_A-405_P10.16mm_Horizontal")
     )
+    (path "/53c4edbd-7c9e-44b0-b5cc-3a777545e753"
+      (reference "H1") (unit 1) (value "MountingHole") (footprint "MountingHole:MountingHole_4.3mm_M4")
+    )
+    (path "/e1792a67-ce3f-4ef4-88e4-0f5af5cc0b53"
+      (reference "H2") (unit 1) (value "MountingHole") (footprint "MountingHole:MountingHole_4.3mm_M4")
+    )
+    (path "/4a0d77ce-560a-47ff-ac64-f3ae2cd334f4"
+      (reference "H3") (unit 1) (value "MountingHole") (footprint "MountingHole:MountingHole_4.3mm_M4")
+    )
+    (path "/4d27752c-ec72-4595-bc74-bb0842d0429a"
+      (reference "H4") (unit 1) (value "MountingHole") (footprint "MountingHole:MountingHole_4.3mm_M4")
+    )
     (path "/ee4fcd98-c198-443e-82b7-b1a28fb4f62d"

Commit message: GERBER
Changed lines of the file:
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@@
     (pin "2")
+  )
+  (symbol (lib_id "MyLib:LOGO") (at 185.42 173.99 0) (unit 1)
+    (in_bom yes) (on_board yes) (fields_autoplaced)
+    (property "Reference" "#G?" (id 0) (at 185.42 167.6287 0)
+      (effects (font (size 1.27 1.27)) hide)
+    )
+    (property "Value" "LOGO" (id 1) (at 185.42 180.3513 0)
+      (effects (font (size 1.27 1.27)) hide)
+    )
+    (property "Footprint" "" (id 2) (at 185.42 173.99 0)
+      (effects (font (size 1.27 1.27)) hide)
+    )
+    (property "Datasheet" "" (id 3) (at 185.42 173.99 0)
+      (effects (font (size 1.27 1.27)) hide)
+    )
   )
   (symbol (lib_id "Device:R") (at 127 77.47 90) (unit 1)
@@
   )
   (symbol_instances
+    (path "/7825e178-7e2e-4378-b0c4-c2033ad1f5ad"
+      (reference "#G?") (unit 1) (value "LOGO") (footprint "")
+    )
     (path "/136436ce-da99-4e2f-834c-0704190d9127"
       (reference "#PWR0101") (unit 1) (value "+5V") (footprint "")
